File: tenax.kicad_pcb (KiCad board)
At the start: 2 copper layers, 247.9 x 99.3 mm, 6 parts, among them J1 MJ-4PP-9, U1 BlackPill

Commit message: Last detais
Parts:
- removed the J1 at (146.3, 102.2)
- removed the J1 at (146.7, 102.2)
- removed REF** (x2): Breakaway_Tabs, teclassio:Breakaway_Tabs
- removed the U1 at (135.7, 72.4)
- removed the U1 at (157.3, 72.4)
- added H1: Breakaway Tabs, tenax:Breakaway_Tabs, F.Cu at (151.6, 65.6)
- added H10: MountingHole, tenax:M2_HOLE_v2, F.Cu at (176.5, 122.4)
- added H11: MountingHole, tenax:M2_HOLE_v2, F.Cu at (111.1, 76.6)
- added H12: MountingHole, tenax:M2_HOLE_v2, F.Cu at (52.6, 106.3)
- added H2: Breakaway Tabs, tenax:Breakaway_Tabs, F.Cu at (151.6, 116.7)
- added H3: MountingHole, tenax:M2_HOLE_v2, F.Cu at (49.3, 87.5)
- added H4: MountingHole, tenax:M2_HOLE_v2, F.Cu at (250.6, 106.3)
- added H5: MountingHole, tenax:M2_HOLE_v2, F.Cu at (218.4, 114.3)
- added H6: MountingHole, tenax:M2_HOLE_v2, F.Cu at (253.9, 87.5)
- added H7: MountingHole, tenax:M2_HOLE_v2, F.Cu at (126.7, 122.4)
- added H8: MountingHole, tenax:M2_HOLE_v2, F.Cu at (84.7, 114.3)
- added H9: MountingHole, tenax:M2_HOLE_v2, F.Cu at (192.0, 76.6)
- added J1: AudioJack4, tenax:MJ-4PP-9_1side, F.Cu at (151.4, 116.7)
- added J2: AudioJack4, tenax:MJ-4PP-9_1side, F.Cu at (151.8, 116.7)
- added SW1: SW_SPST, tenax:CherryMX_Hotswap, F.Cu at (38.2, 79.8)
- added SW10: SW_SPST, tenax:CherryMX_Hotswap, F.Cu at (93.7, 124.3)
- added SW11: SW_SPST, tenax:CherryMX_Hotswap, F.Cu at (101.6, 67.1)
- added SW12: SW_SPST, tenax:CherryMX_Hotswap, F.Cu at (101.6, 86.1)
- added SW13: SW_SPST, tenax:CherryMX_Hotswap, F.Cu at (101.6, 105.2)
- added SW14: SW_SPST, tenax:CherryMX_Hotswap, F.Cu at (114.6, 128.4)
- added SW15: SW_SPST, tenax:CherryMX_Hotswap, F.Cu at (120.6, 69.6)
- added SW16: SW_SPST, tenax:CherryMX_Hotswap, F.Cu at (120.6, 88.6)
- added SW17: SW_SPST, tenax:CherryMX_Hotswap, F.Cu at (120.6, 107.7)
- added SW18: SW_SPST, tenax:CherryMX_Hotswap, F.Cu at (133.8, 137.8)
- added SW19: SW_SPST, tenax:CherryMX_Hotswap, F.Cu at (182.5, 69.6)
- added SW2: SW_SPST, tenax:CherryMX_Hotswap, F.Cu at (41.5, 98.6)
- added SW20: SW_SPST, tenax:CherryMX_Hotswap, F.Cu at (182.5, 88.6)
- added SW21: SW_SPST, tenax:CherryMX_Hotswap, F.Cu at (182.5, 107.7)
- added SW22: SW_SPST, tenax:CherryMX_Hotswap, F.Cu at (169.3, 137.8)
- added SW23: SW_SPST, tenax:CherryMX_Hotswap, F.Cu at (201.5, 67.1)
- added SW24: SW_SPST, tenax:CherryMX_Hotswap, F.Cu at (201.5, 86.1)
- added SW25: SW_SPST, tenax:CherryMX_Hotswap, F.Cu at (201.5, 105.2)
- added SW26: SW_SPST, tenax:CherryMX_Hotswap, F.Cu at (188.5, 128.4)
- added SW27: SW_SPST, tenax:CherryMX_Hotswap, F.Cu at (220.6, 60.6)
- added SW28: SW_SPST, tenax:CherryMX_Hotswap, F.Cu at (220.6, 79.6)
- added SW29: SW_SPST, tenax:CherryMX_Hotswap, F.Cu at (220.6, 98.7)
- added SW3: SW_SPST, tenax:CherryMX_Hotswap, F.Cu at (44.8, 117.3)
- added SW30: SW_SPST, tenax:CherryMX_Hotswap, F.Cu at (209.5, 124.3)
- added SW31: SW_SPST, tenax:CherryMX_Hotswap, F.Cu at (239.6, 66.6)
- added SW32: SW_SPST, tenax:CherryMX_Hotswap, F.Cu at (239.6, 85.6)
- added SW33: SW_SPST, tenax:CherryMX_Hotswap, F.Cu at (239.6, 104.7)
- added SW34: SW_SPST, tenax:CherryMX_Hotswap, F.Cu at (264.9, 79.8)
- added SW35: SW_SPST, tenax:CherryMX_Hotswap, F.Cu at (261.6, 98.6)
- added SW36: SW_SPST, tenax:CherryMX_Hotswap, F.Cu at (258.3, 117.3)
- added SW4: SW_SPST, tenax:CherryMX_Hotswap, F.Cu at (63.5, 66.6)
- added SW5: SW_SPST, tenax:CherryMX_Hotswap, F.Cu at (63.5, 85.6)
- added SW6: SW_SPST, tenax:CherryMX_Hotswap, F.Cu at (63.5, 104.7)
- added SW7: SW_SPST, tenax:CherryMX_Hotswap, F.Cu at (82.5, 60.6)
- added SW8: SW_SPST, tenax:CherryMX_Hotswap, F.Cu at (82.5, 79.6)
- added SW9: SW_SPST, tenax:CherryMX_Hotswap, F.Cu at (82.5, 98.7)
- added U1: YAAJ_WeAct_BlackPill_Part_Like, tenax:BlackPill_STLINK, B.Cu at (140.8, 86.8)
- added U2: YAAJ_WeAct_BlackPill_Part_Like, tenax:BlackPill_STLINK, B.Cu at (162.4, 86.8)
Routing:
- net +3V3: track 0.00 -> 136.2 mm
- net /k2_0: track 0.00 -> 135.2 mm
- net /k2_9: track 0.00 -> 121.3 mm
- net /k2_1: track 0.00 -> 119.7 mm
- net /k0_0: track 0.00 -> 118.6 mm
- net /k1_0: track 0.00 -> 107.2 mm
- net /k2_8: track 0.00 -> 107.0 mm
- net /k2_2: track 0.00 -> 105.0 mm
- net /k2_7: track 0.00 -> 96.2 mm
- net /k2_3: track 0.00 -> 95.1 mm
- net /k1_9: track 0.00 -> 92.1 mm
- net /k0_9: track 0.00 -> 91.4 mm
- net /k0_1: track 0.00 -> 86.7 mm
- net /k1_1: track 0.00 -> 83.2 mm
- net /k3_0: track 0.00 -> 79.7 mm
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- added copper zone on B.Cu, net GND
- added copper zone on F.Cu, net GND
Other:
- board size 247.9 x 99.3 mm -> 248.4 x 99.5 mm
